File: src/libs/core/layouts/default/default.kicad_pcb (KiCad board)
At the start: 2 copper layers, 0 parts

Commit message: good base
Parts:
- added C1: 100nF ±10% 16V X7R, Samsung_Electro_Mechanics_CL05B104KO5NNNC:C0402, F.Cu at (143.9, 46.3)
- added C2: 100nF ±10% 16V X7R, Samsung_Electro_Mechanics_CL05B104KO5NNNC:C0402, F.Cu at (143.9, 29.3)
- added C3: 22µF ±20% 6.3V X5R, Samsung_Electro_Mechanics_CL10A226MQ8NRNC:C0603, F.Cu at (154.2, 28.8)
- added C4: 100nF ±10% 16V X7R, Samsung_Electro_Mechanics_CL05B104KO5NNNC:C0402, F.Cu at (153.4, 30.3)
- added C5: 10µF ±10% 25V X5R, Samsung_Electro_Mechanics_CL21A106KAYNNNE:C0805, F.Cu at (142.2, 22.6)
- added C6: 22µF ±20% 6.3V X5R, Samsung_Electro_Mechanics_CL21A226MQQNNNE:C0805, F.Cu at (154.0, 20.2)
- added C8: 100nF ±10% 16V X7R, Samsung_Electro_Mechanics_CL05B104KO5NNNC:C0402, F.Cu at (140.6, 44.6)
- added C9: 100nF ±10% 16V X7R, Samsung_Electro_Mechanics_CL05B104KO5NNNC:C0402, F.Cu at (130.9, 25.9)
- added CN1: , JST_Sales_America_BM04B_SRSS_TB_LF__SN:CONN-SMD_BM04B-SRSS-TB, F.Cu at (138.0, 39.8)
- added D1: , STMicroelectronics_USBLC6_2SC6:SOT-23-6_L2.9-W1.6-P0.95-LS2.8-BL, F.Cu at (133.2, 25.2)
- added F1: , BHFUSE_BSMD0805_050_15V:F0805, F.Cu at (137.2, 24.9)
- added LED1: , OPSCO_SK6805_EC20:LED-SMD_4P-L2.0-W2.0-BR, F.Cu at (140.7, 46.6)
- added LED2: , Lite_On_LTST_C191KGKT:LED0603-RD, F.Cu at (141.6, 30.4)
- added R1: 4.7kΩ ±1% 62.5mW, UNI_ROYAL_0402WGF4701TCE:R0402, F.Cu at (142.0, 38.2)
- added R10: 1kΩ ±1% 62.5mW, UNI_ROYAL_0402WGF1001TCE:R0402, F.Cu at (116.9, 27.2)
- added R11: 1kΩ ±1% 62.5mW, UNI_ROYAL_0402WGF1001TCE:R0402, F.Cu at (114.4, 27.3)
- added R12: 1kΩ ±1% 62.5mW, UNI_ROYAL_0402WGF1001TCE:R0402, F.Cu at (111.9, 27.3)
- added R13: 1kΩ ±1% 62.5mW, UNI_ROYAL_0402WGF1001TCE:R0402, F.Cu at (105.9, 27.2)
- added R14: 1kΩ ±1% 62.5mW, UNI_ROYAL_0402WGF1001TCE:R0402, F.Cu at (103.4, 27.2)
- added R15: 1kΩ ±1% 62.5mW, UNI_ROYAL_0402WGF1001TCE:R0402, F.Cu at (100.9, 27.3)
- added R16: 1kΩ ±1% 62.5mW, UNI_ROYAL_0402WGF1001TCE:R0402, F.Cu at (98.4, 27.3)
- added R2: 4.7kΩ ±1% 62.5mW, UNI_ROYAL_0402WGF4701TCE:R0402, F.Cu at (142.0, 39.6)
- added R3: 10kΩ ±1% 62.5mW, UNI_ROYAL_0402WGF1002TCE:R0402, F.Cu at (152.0, 28.7)
- added R4: 10kΩ ±1% 62.5mW, UNI_ROYAL_0402WGF1002TCE:R0402, F.Cu at (143.9, 41.4)
- added R5: 10kΩ ±1% 62.5mW, UNI_ROYAL_0402WGF1002TCE:R0402, F.Cu at (150.8, 28.7)
- added R6: 1kΩ ±1% 62.5mW, UNI_ROYAL_0402WGF1001TCE:R0402, F.Cu at (140.4, 30.8)
- added R7: 5.1kΩ ±1% 62.5mW, UNI_ROYAL_0402WGF5101TCE:R0402, F.Cu at (135.4, 25.2)
- added R8: 5.1kΩ ±1% 62.5mW, UNI_ROYAL_0402WGF5101TCE:R0402, F.Cu at (129.7, 25.2)
- added R9: 1kΩ ±1% 62.5mW, UNI_ROYAL_0402WGF1001TCE:R0402, F.Cu at (119.4, 27.2)
- added SW1: , ALPSALPINE_SKRPACE010:KEY-SMD_4P-L4.2-W3.2-P2.20-LS4.6, F.Cu at (147.4, 46.3)
- added SW2: , ALPSALPINE_SKRPACE010:KEY-SMD_4P-L4.2-W3.2-P2.20-LS4.6, F.Cu at (147.4, 29.3)
- added U1: , Espressif_Systems_ESP32_C3_MINI_1_N4:WIFIM-SMD_ESP32-C3-MINI-1, F.Cu at (150.4, 37.8)
- added U2: , Advanced_Monolithic_Systems_AMS1117_3_3:SOT-223-3_L6.5-W3.4-P2.30-LS7.0-BR, F.Cu at (148.6, 20.2)
- added U3: , HCTL_PM254_2_04_W_8_5:HDR-TH_8P-P2.54-H-F-R2-C4-W8.5, F.Cu at (115.6, 23.8)
- added U4: , HCTL_PM254_2_04_W_8_5:HDR-TH_8P-P2.54-H-F-R2-C4-W8.5, F.Cu at (102.1, 23.8)
- added USB1: , SHOU_HAN_TYPE_C_16PIN_2MD_073:USB-C-SMD_TYPE-C-6PIN-2MD-073, F.Cu at (133.2, 19.4)
Routing:
- net hv-1: track 0.00 -> 25.8 mm, vias 0 -> 1
- net -hv: track 0.00 -> 20.6 mm, vias 0 -> 3
- net gnd: track 0.00 -> 19.9 mm, vias 0 -> 9
- net hv-0: track 0.00 -> 10.6 mm
- net -line-0: track 0.00 -> 10.1 mm
- net -line-1: track 0.00 -> 9.84 mm
- net line-4: track 0.00 -> 7.57 mm
- net line-5: track 0.00 -> 6.68 mm
- net output-0: track 0.00 -> 6.52 mm
- net output-1: track 0.00 -> 5.33 mm
- net line-1: track 0.00 -> 3.66 mm
- net line-0: track 0.00 -> 3.35 mm
- net -line-5: track 0.00 -> 3.10 mm
- net debug_header.headers[0]-_8: track 0.00 -> 1.83 mm
- net debug_header.headers[1]-_8: track 0.00 -> 1.83 mm
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- added copper zone on B.Cu, net gnd
- added copper zone on F.Cu, net gnd
Other:
- board outline added: 24.6 x 8.1 mm
- board text added: "BOARD EDGE"
