File: src/products/espaper/layouts/default/default.kicad_pcb (KiCad board)
At the start: 2 copper layers, 50 x 25 mm, 43 parts

Commit message: almost done, need to finish a few traces
Parts:
- added B1: , EEMB_BATTERY_LP402535:EEMB_BATTERY_LP402535, B.Cu at (148.9, 101.3)
- added C19: 4.7µF ±10% 16V X5R, Samsung_Electro_Mechanics_CL10A475KO8NNNC:C0603, F.Cu at (144.8, 105.5)
- added C20: 22µF ±20% 6.3V X5R, Samsung_Electro_Mechanics_CL21A226MQQNNNE:C0805, F.Cu at (133.3, 113.7)
- added C21: 22µF ±20% 6.3V X5R, Samsung_Electro_Mechanics_CL21A226MQQNNNE:C0805, F.Cu at (133.3, 111.7)
- added C22: 22µF ±20% 6.3V X5R, Samsung_Electro_Mechanics_CL21A226MQQNNNE:C0805, F.Cu at (133.3, 109.7)
- added C23: 22µF ±20% 6.3V X5R, Samsung_Electro_Mechanics_CL21A226MQQNNNE:C0805, F.Cu at (133.3, 107.7)
- added C24: 100nF ±10% 16V X7R, Samsung_Electro_Mechanics_CL05B104KO5NNNC:C0402, F.Cu at (128.8, 106.7)
- added C25: 1µF ±10% 25V X5R, Samsung_Electro_Mechanics_CL05A105KA5NQNC:C0402, F.Cu at (142.0, 101.6)
- added C26: 10µF ±20% 6.3V X5R, Murata_Electronics_GRM155R60J106ME44D:C0402, F.Cu at (143.7, 100.3)
- added C27: 1µF ±10% 25V X5R, Samsung_Electro_Mechanics_CL05A105KA5NQNC:C0402, F.Cu at (146.3, 100.3)
- added L1: 1µH ±20% 4.7A 18mΩ, cjiang_FNR4030S1R0MT:IND-SMD_L4.0-W4.0_FNR40XXS, F.Cu at (136.3, 103.7)
- added R15: 2kΩ ±1% 62.5mW, UNI_ROYAL_0402WGF2001TCE:R0402, F.Cu at (148.0, 101.9)
- added R16: 10kΩ ±1% 62.5mW, UNI_ROYAL_0402WGF1002TCE:R0402, F.Cu at (142.0, 102.8)
- added R17: 18kΩ ±1% 62.5mW, UNI_ROYAL_0402WGF1802TCE:R0402, F.Cu at (148.0, 102.9)
- added R18: 10kΩ ±1% 62.5mW, UNI_ROYAL_0402WGF1002TCE:R0402, F.Cu at (145.0, 96.1)
- added R19: 10kΩ ±1% 62.5mW, UNI_ROYAL_0402WGF1002TCE:R0402, F.Cu at (146.7, 103.9)
- added U3: , Texas_Instruments_TPS63020DSJR:VSON-14_L4.0-W3.0-P0.50-BL-EP_TI_DSJ, F.Cu at (131.6, 103.7)
- added U4: , BQ25185DLHR_BQ25185DLHR:WSON-10_L2.2-W2.0-P0.40-BL-EP_TI_DLH0010A, F.Cu at (145.0, 102.2)
- C3, C4: value 1µF ±10% 25V X5R -> 10µF ±10% 25V X5R; footprint Samsung_Electro_Mechanics_CL05A105KA5NQNC:C0402 -> Samsung_Electro_Mechanics_CL21A106KAYNNNE:C0805
- R1: value 10kΩ ±1% 62.5mW -> 180kΩ ±1% 62.5mW; footprint UNI_ROYAL_0402WGF1002TCE:R0402 -> UNI_ROYAL_0402WGF1803TCE:R0402
- R2: value 18kΩ ±1% 62.5mW -> 1MΩ ±1% 62.5mW; footprint UNI_ROYAL_0402WGF1802TCE:R0402 -> UNI_ROYAL_0402WGF1004TCE:R0402
- R3: value 10kΩ ±1% 62.5mW -> 3.3Ω ±1% 62.5mW; footprint UNI_ROYAL_0402WGF1002TCE:R0402 -> UNI_ROYAL_0402WGF330KTCE:R0402
- R5: value 10kΩ ±1% 62.5mW -> 1MΩ ±1% 62.5mW; footprint UNI_ROYAL_0402WGF1002TCE:R0402 -> UNI_ROYAL_0402WGF1004TCE:R0402
- U1: footprint STMicroelectronics_LDK220M_R:SOT-23-5_L3.0-W1.7-P0.95-LS2.8-BL -> MOLEX_532610271:CONN-SMD_532610271
- moved R5 25.3 mm to (130.1, 99.7), turned to 90 degrees
- moved R12 13.6 mm to (154.5, 92.9)
- moved R7 10.3 mm to (168.8, 105.5)
- moved R9 10.3 mm to (168.8, 104.3)
- moved C14 10.3 mm to (151.2, 97.4)
- moved C15 10.3 mm to (168.2, 97.4)
- moved C16 10.3 mm to (168.7, 107.7)
- moved C17 10.3 mm to (167.2, 106.9)
- moved R8 10.3 mm to (156.1, 97.4)
- moved SW1 10.3 mm to (151.2, 100.9)
- moved SW2 10.3 mm to (168.2, 100.9)
- moved U2 10.3 mm to (159.7, 103.9)
- moved U1 10.3 mm to (131.9, 92.4), turned to 90 degrees
- moved R2 9.20 mm to (130.8, 108.7), turned to 90 degrees
- moved R1 8.87 mm to (130.3, 107.2), turned to 180 degrees
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Connections:
- C1 pad 1: -hv-0 -> -hv-1
- C10 pad 1: -line-7 -> cathode
- C11 pad 1: -line-8 -> -line-9
- C13 pad 1: -line-9 -> -line-10
- C16 pad 1: -hv-0 -> -hv-1
- C17 pad 1: -hv-0 -> -hv-1
- C3 pad 1: -hv-1 -> VIN
- C4 pad 1: -hv-0 -> VIN
- C5 pad 1: -line-3 -> -line-4
- C6 pad 1: cathode -> -line-5
- C7 pad 1: -line-4 -> -line-6
- C8 pad 1: -line-5 -> -line-7
- C9 pad 1: -line-6 -> -line-8
- FPC1 pad 10: -line-12 -> -line-11
- FPC1 pad 11: -line-2 -> -line-3
- FPC1 pad 12: output-0 -> -line-2
- FPC1 pad 13: -line-13 -> -line-12
- FPC1 pad 14: -line-14 -> -line-13
- FPC1 pad 16: -hv-0 -> -hv-1
- FPC1 pad 18: -line-4 -> -line-6
- FPC1 pad 19: -line-5 -> -line-7
- FPC1 pad 20: -line-6 -> -line-8
- FPC1 pad 21: -line-7 -> cathode
- FPC1 pad 22: -line-8 -> -line-9
- FPC1 pad 24: -line-9 -> -line-10
- FPC1 pad 4: -line-3 -> -line-4
- FPC1 pad 5: cathode -> -line-5
- L2 pad 1: -hv-0 -> -hv-1
- R1 pad 1: ADJ_NC -> FB
- R12 pad 1: -line-12 -> -line-11
- R12 pad 2: -hv-0 -> -hv-1
- R2 pad 1: -hv-0 -> -hv-1
- R2 pad 2: ADJ_NC -> FB
- R4 pad 2: -hv-0 -> -hv-1
- R5 pad 1: output-0 -> PG
- R5 pad 2: -hv-0 -> -hv-1
- R6 pad 1: -line-2 -> -line-3
- R6 pad 2: -hv-0 -> -hv-1
- R7 pad 1: -line-10 -> -line-1
- R7 pad 2: -hv-0 -> -hv-1
- R8 pad 1: -line-15 -> -line-14
- R8 pad 2: -hv-0 -> -hv-1
- R9 pad 1: -hv-0 -> -hv-1
- U1 pad 1: -hv-1 -> gnd
- U1 pad 2: gnd -> -hv-0
- U1 pad 3: -hv-1 -> gnd
- U1 pad 4: ADJ_NC -> gnd
- U2 pad 16: -line-13 -> -line-12
- U2 pad 18: -line-11 -> -line-3
- U2 pad 21: -line-14 -> -line-13
- U2 pad 22: -line-15 -> -line-14
- U2 pad 26: -line-17 -> -line-15
- U2 pad 27: -line-18 -> -line-16
- U2 pad 3: -hv-0 -> -hv-1
- U2 pad 5: -line-10 -> -line-1
- U2 pad 6: -line-16 -> -line-11
- USB1 pad A4: -hv-1 -> -hv-2
- USB1 pad A6: -line-18 -> -line-16
- USB1 pad A7: -line-17 -> -line-15
- USB1 pad A9: -hv-1 -> -hv-2
- USB1 pad B4: -hv-1 -> -hv-2
- USB1 pad B6: -line-18 -> -line-16
- USB1 pad B7: -line-17 -> -line-15
- USB1 pad B9: -hv-1 -> -hv-2
Routing:
- net -hv-1: track 4.83 -> 80.2 mm, vias 0 -> 4
- net gnd: track 12.6 -> 49.9 mm, vias 0 -> 25
- net -anode-1: track 0.00 -> 37.1 mm
- net cathode: track 0.00 -> 36.8 mm
- net -line-15: track 1.61 -> 22.2 mm
- net -line-16: track 0.00 -> 19.9 mm
- net VIN: track 0.00 -> 19.3 mm, vias 0 -> 4
- net -hv-2: track 0.00 -> 13.3 mm
- net source: track 0.00 -> 12.7 mm
- net EN: track 0.00 -> 11.8 mm, vias 0 -> 2
- net gate: track 0.00 -> 11.0 mm
- net -hv-0: track 9.34 -> 17.3 mm
- net -line-1: track 0.00 -> 6.65 mm, vias 0 -> 2
- net sw_node: track 0.00 -> 6.05 mm
- net -line-11: track 0.00 -> 5.55 mm, vias 0 -> 2
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- added copper zone on F.Cu, net (none)
- added copper zone on F.Cu, net -hv-1
- added copper zone on F.Cu, net -hv-2
- added copper zone on F.Cu, net L1
- added copper zone on F.Cu, net L2
- added copper zone on F.Cu, net VIN
- added copper zone on B.Cu, net gnd
Other:
- board size 50 x 25 mm -> 41.8 x 27 mm
- board text added: "+"
- board text added: "-"

Commit message: shipped espaper on jlc
Parts:
- added LED1: , Hubei_KENTO_Elec_Blue_light_0603:LED0603-RD, F.Cu at (163.4, 97.4)
- added LED2: , Hubei_KENTO_Elec_KT_0603R:LED0603-RD, F.Cu at (128.9, 99.5)
- added LOGO1: , atopile_Logo_4x4mm:atopile_Logo_4x4mm, F.Cu at (149.2, 112.5)
- added R20: 10kΩ ±1% 62.5mW, UNI_ROYAL_0402WGF1002TCE:R0402, F.Cu at (166.0, 97.4)
- added R21: 10kΩ ±1% 62.5mW, UNI_ROYAL_0402WGF1002TCE:R0402, F.Cu at (130.3, 97.4)
- L2: value 68µH ±10% 9MHz 2mA 2Ω -> 68µH ±20% 50mA 6Ω; footprint TDK_MLF2012C680KT000:L0805 -> Taiyo_Yuden_LB2012T680M:L0805
- R1: value 180kΩ ±1% 62.5mW -> 200kΩ ±1% 62.5mW; footprint UNI_ROYAL_0402WGF1803TCE:R0402 -> UNI_ROYAL_0402WGF2003TCE:R0402
- R10: value 470mΩ ±1% 62.5mW -> 470mΩ ±1%; footprint UNI_ROYAL_0402WGF470LTCE:R0402 -> YAGEO_RL0402FR_070R47L:R0402
- R17: footprint UNI_ROYAL_0402WGF1802TCE:R0402 -> YAGEO_RC0402FR_0718KL:R0402
- R2: value 1MΩ ±1% 62.5mW -> 1.2MΩ ±1% 62.5mW; footprint UNI_ROYAL_0402WGF1004TCE:R0402 -> FOJAN_FRC0402F1204TS:R0402
- moved R6 7.85 mm to (160.1, 97.4), turned to 90 degrees
- moved C10 0.44 mm to (139.2, 99.4)
- moved D2 0.40 mm to (164.3, 91.7)
- moved D3 0.20 mm to (164.6, 93.6)
- moved R18 0.10 mm to (145.0, 96.2)
- moved C9 0.09 mm to (140.6, 96.6)
Connections:
- net -anode-0 renamed d_gnd-anode
- net -anode-1 renamed prevgl-anode
- net -hv-0 renamed power-VCC
- net -hv-2 renamed POWER_VBUS
- net -line-0 renamed bs-line
- net -line-1 renamed EPD_BUSY
- net -line-10 renamed vcom-line
- net -line-11 renamed EPD_RST
- net -line-12 renamed EPD_SPI_SCLK
- net -line-13 renamed EPD_SPI_MOSI
- net -line-14 renamed EPD_SPI_MISO
- net -line-15 renamed USB_D_N
- net -line-16 renamed USB_D_P
- net -line-2 renamed EPD_SPI_CS
- net -line-3 renamed EPD_DC
- net -line-4 renamed vgl-line
- net -line-5 renamed vgh-line
- net -line-6 renamed vdd-line
- net -line-7 renamed vpp-line
- net -line-8 renamed vsh-line
- net -line-9 renamed vsl-line
- net EN renamed _power_in_a-VCC
- net FB renamed VDIV_OUTPUT
- net VIN renamed power_sys-VCC
- net cathode renamed prevgh-cathode
- net epd_fpc-line-0 renamed hlt_ctl-line
- net epd_fpc-line-1 renamed tscl-line
- net epd_fpc-line-2 renamed tsda-line
- net esp32-line-0 renamed SCK
- net esp32-line-2 renamed data_2
- net esp32-line-3 renamed RX
- net esp32-line-4 renamed TX
- net esp32-line-5 renamed SCL
- net esp32.esp32_c3.package.footprint.pins[16].net-net renamed esp32-net-0
- net esp32.esp32_c3.package.footprint.pins[17].net-net renamed esp32-net-1
- net esp32.esp32_c3.package.footprint.pins[1].net-net renamed esp32-net-2
- net esp32.esp32_c3.package.footprint.pins[20].net-net renamed esp32-net-3
- net esp32.esp32_c3.package.footprint.pins[21].net-net renamed esp32-net-4
- net esp32.esp32_c3.package.footprint.pins[25].net-net renamed esp32-net-5
- net esp32.esp32_c3.package.footprint.pins[26].net-net renamed esp32-net-6
- net esp32.esp32_c3.package.footprint.pins[27].net-net renamed esp32-net-7
- net esp32.esp32_c3.package.footprint.pins[28].net-net renamed esp32-net-8
- net esp32.esp32_c3.package.footprint.pins[33].net-net renamed esp32-net-9
- net esp32.esp32_c3.package.footprint.pins[50].net-net renamed esp32-net-10
- net esp32.esp32_c3.package.footprint.pins[52].net-net renamed esp32-net-11
- net esp32.esp32_c3.package.footprint.pins[6].net-net renamed esp32-net-12
- net esp32.esp32_c3.package.footprint.pins[8].net-net renamed esp32-net-13
- net output-0 renamed output
- net output-1 renamed N_TRST
- net sw_node renamed charge_pump_inductor-anode
- net usb.conn.footprint.pins[0].net-net renamed conn-net
- C1 pad 1: -hv-1 -> POWER_3V3
- C1 pad 2: gnd -> model-power-GND
- C10 pad 2: gnd -> model-power-GND
- C11 pad 2: gnd -> model-power-GND
- C12 pad 2: gnd -> model-power-GND
- C13 pad 2: gnd -> model-power-GND
- C14 pad 1: gnd -> model-power-GND
- C15 pad 1: gnd -> model-power-GND
- C16 pad 1: -hv-1 -> POWER_3V3
- C16 pad 2: gnd -> model-power-GND
- C17 pad 1: -hv-1 -> POWER_3V3
- C17 pad 2: gnd -> model-power-GND
- C19 pad 2: gnd -> model-power-GND
- C2 pad 2: gnd -> model-power-GND
- C20 pad 1: -hv-1 -> POWER_3V3
- C20 pad 2: gnd -> model-power-GND
- C21 pad 1: -hv-1 -> POWER_3V3
- C21 pad 2: gnd -> model-power-GND
- C22 pad 1: -hv-1 -> POWER_3V3
- C22 pad 2: gnd -> model-power-GND
- C23 pad 1: -hv-1 -> POWER_3V3
- C23 pad 2: gnd -> model-power-GND
- C24 pad 2: gnd -> model-power-GND
- C25 pad 2: gnd -> model-power-GND
- C26 pad 2: gnd -> model-power-GND
- C27 pad 2: gnd -> model-power-GND
- C3 pad 2: gnd -> model-power-GND
- C4 pad 2: gnd -> model-power-GND
- C5 pad 2: gnd -> model-power-GND
- C6 pad 2: gnd -> model-power-GND
- C7 pad 2: gnd -> model-power-GND
- C8 pad 2: gnd -> model-power-GND
- C9 pad 2: gnd -> model-power-GND
- D1 pad 1: gnd -> model-power-GND
- FPC1 pad 16: -hv-1 -> POWER_3V3
- FPC1 pad 17: gnd -> model-power-GND
- L2 pad 1: -hv-1 -> POWER_3V3
- R1 pad 2: gnd -> model-power-GND
- R10 pad 2: gnd -> model-power-GND
- R11 pad 2: gnd -> model-power-GND
- R12 pad 2: -hv-1 -> POWER_3V3
- R13 pad 2: gnd -> model-power-GND
- R14 pad 2: gnd -> model-power-GND
- R15 pad 2: gnd -> model-power-GND
- R16 pad 2: gnd -> model-power-GND
- R17 pad 2: gnd -> model-power-GND
- R18 pad 2: gnd -> POWER_3V3
- R19 pad 2: gnd -> model-power-GND
- R2 pad 1: -hv-1 -> POWER_3V3
- R3 pad 2: gnd -> model-power-GND
- R4 pad 2: -hv-1 -> POWER_3V3
- R5 pad 2: -hv-1 -> POWER_3V3
- R6 pad 2: -hv-1 -> POWER_3V3
- R7 pad 2: -hv-1 -> POWER_3V3
- R8 pad 2: -hv-1 -> POWER_3V3
- R9 pad 1: -hv-1 -> POWER_3V3
- SW1 pad 1: gnd -> model-power-GND
- SW1 pad 2: gnd -> model-power-GND
- SW2 pad 1: gnd -> model-power-GND
- SW2 pad 2: gnd -> model-power-GND
- U1 pad 1: gnd -> model-power-GND
- U1 pad 3: gnd -> model-power-GND
- U1 pad 4: gnd -> model-power-GND
- U2 pad 1: gnd -> model-power-GND
- U2 pad 11: gnd -> model-power-GND
- U2 pad 13: esp32-line-1 -> power-anode
- U2 pad 14: gnd -> model-power-GND
- U2 pad 2: gnd -> model-power-GND
- U2 pad 3: -hv-1 -> POWER_3V3
- U2 pad 36: gnd -> model-power-GND
- U2 pad 37: gnd -> model-power-GND
- U2 pad 38: gnd -> model-power-GND
- U2 pad 39: gnd -> model-power-GND
- U2 pad 40: gnd -> model-power-GND
- U2 pad 41: gnd -> model-power-GND
- U2 pad 42: gnd -> model-power-GND
- U2 pad 43: gnd -> model-power-GND
- U2 pad 44: gnd -> model-power-GND
- U2 pad 45: gnd -> model-power-GND
- U2 pad 46: gnd -> model-power-GND
- U2 pad 47: gnd -> model-power-GND
- U2 pad 48: gnd -> model-power-GND
- U2 pad 49: gnd -> model-power-GND
- U2 pad 50: gnd -> model-power-GND
- U2 pad 51: gnd -> model-power-GND
- U2 pad 52: gnd -> model-power-GND
- U2 pad 53: gnd -> model-power-GND
- U3 pad 15: gnd -> model-power-GND
- U3 pad 2: gnd -> model-power-GND
- U3 pad 4: -hv-1 -> POWER_3V3
- U3 pad 5: -hv-1 -> POWER_3V3
- U4 pad 11: gnd -> model-power-GND
- U4 pad 3: STAT2 -> red_led-power-GND
- U4 pad 5: gnd -> model-power-GND
- USB1 pad 1: gnd -> model-power-GND
- USB1 pad 2: gnd -> model-power-GND
- USB1 pad 3: gnd -> model-power-GND
- USB1 pad 4: gnd -> model-power-GND
- USB1 pad A1: gnd -> model-power-GND
- USB1 pad A12: gnd -> model-power-GND
- USB1 pad B1: gnd -> model-power-GND
- USB1 pad B12: gnd -> model-power-GND
Routing:
- net POWER_3V3: track 0.00 -> 138.4 mm, vias 0 -> 6
- net -hv-1: track 80.2 -> 0.00 mm, vias 4 -> 0
- net model-power-GND: track 0.00 -> 73.5 mm, vias 0 -> 43
- net gnd: track 49.9 -> 0.00 mm, vias 25 -> 0
- net EPD_RST: track 5.55 -> 35.6 mm, vias 2 -> 3
- net EPD_BUSY: track 6.65 -> 36.3 mm, vias 2 -> 3
- net EPD_SPI_SCLK: track 2.68 -> 26.9 mm, vias 1 -> 2
- net EPD_DC: track 1.78 -> 23.5 mm, vias 1 -> 2
- net EPD_SPI_MOSI: track 3.87 -> 25.2 mm, vias 1 -> 2
- net red_led-power-GND: track 0.00 -> 16.7 mm, vias 0 -> 2
- net POWER_VBUS: track 13.3 -> 23.0 mm
- net bs-line: track 3.71 -> 10.5 mm, vias 1 -> 2
- net conn-net: track 0.00 -> 6.20 mm
- net USB_D_P: track 19.9 -> 22.9 mm, vias 0 -> 2
- net power-anode: track 0.00 -> 2.06 mm
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- added copper zone on F.Cu, net POWER_3V3
- added copper zone on B.Cu, net model-power-GND
- added copper zone on F.Cu, net model-power-GND
- removed copper zone on F.Cu, net -hv-1
- removed copper zone on B.Cu, net gnd
- removed copper zone on F.Cu, net gnd
Other:
- board size 41.8 x 27 mm -> 42 x 27 mm
- board text added: "CHG"
- board text added: "atopile"
- board text added: "espaper display"
